Commit message: [modify] regenerate fr01.urdf

File: fr01_description/robots/urdf/fr01.urdf (robot description, URDF)
Before this commit: robot fr01, 16 links, 15 joints
Links:
- removed link support_left_back_link
- removed link support_left_front_link
- removed link support_right_back_link
- removed link support_right_front_link
- added link steer_left_back_link, mass 2.522; collision mesh filename=package://fr01_description/meshes/collision/steer_link.stl; visual mesh filename=package://fr01_description/meshes/visual/steer_link.dae
- added link steer_left_front_link, mass 2.522; collision mesh filename=package://fr01_description/meshes/collision/steer_link.stl; visual mesh filename=package://fr01_description/meshes/visual/steer_link.dae
- added link steer_right_back_link, mass 2.522; collision mesh filename=package://fr01_description/meshes/collision/steer_link.stl; visual mesh filename=package://fr01_description/meshes/visual/steer_link.dae
- added link steer_right_front_link, mass 2.522; collision mesh filename=package://fr01_description/meshes/collision/steer_link.stl; visual mesh filename=package://fr01_description/meshes/visual/steer_link.dae
Joints:
- removed joint support_left_back_joint
- removed joint support_left_front_joint
- removed joint support_right_back_joint
- removed joint support_right_front_joint
- added joint steer_left_back_joint: type revolute, parent rocker_left_link, child steer_left_back_link, origin xyz=-0.4 0.05 -0.1 rpy=0 0 -1.57079637, axis 0 0 1, limit lower=-1.57079637 upper=1.57079637 effort=30.0 velocity=6.28318548
- added joint steer_left_front_joint: type revolute, parent bogie_left_link, child steer_left_front_link, origin xyz=-0.202 -0.115 0.05 rpy=0 0 1.57079637, axis 0 0 1, limit lower=-1.57079637 upper=1.57079637 effort=30.0 velocity=6.28318548
- added joint steer_right_back_joint: type revolute, parent rocker_right_link, child steer_right_back_link, origin xyz=-0.4 -0.05 -0.1 rpy=0 0 1.57079637, axis 0 0 1, limit lower=-1.57079637 upper=1.57079637 effort=30.0 velocity=6.28318548
- added joint steer_right_front_joint: type revolute, parent bogie_right_link, child steer_right_front_link, origin xyz=-0.202 0.115 0.05 rpy=0 0 -1.57079637, axis 0 0 1, limit lower=-1.57079637 upper=1.57079637 effort=30.0 velocity=6.28318548
- joint wheel_left_back_joint: parent support_left_back_link -> steer_left_back_link
- joint wheel_left_front_joint: parent support_left_front_link -> steer_left_front_link
- joint wheel_right_back_joint: parent support_right_back_link -> steer_right_back_link
- joint wheel_right_front_joint: parent support_right_front_link -> steer_right_front_link
