Commit message: [modify] set back dynamics values of passive joints to its original ones.

File: fr01_description/urdf/leg/leg.urdf.xacro (robot description, xacro)
@@ -9,5 +9,5 @@
 	  <child link="bogie_${side}_link"/>
 	  <insert_block name="joint_axis"/>
-	  <dynamics dampint="0.04" friction="0.01"/>
+	  <dynamics dampint="0.7" friction="0.7"/>
 	  <limit effort="30.0" lower="${-M_PI/2}" upper="${M_PI/2}" velocity="${2*M_PI}"/>
 	</joint>
@@ -37,5 +37,5 @@
 	  <child link="rocker_${side}_link"/>
 	  <insert_block name="joint_axis"/>
-	  <dynamics dampint="1.4" friction="1.0"/>
+	  <dynamics dampint="0.7" friction="0.7"/>
 	  <limit effort="30.0" lower="${-M_PI/2}" upper="${M_PI/2}" velocity="${2*M_PI}"/>
 	</joint>
