Commit message: [modify] modify the xacro files
use the insert_block macros

File: fr01_description/robots/fr01.urdf.xacro (robot description, xacro)
@@ -10,5 +10,5 @@
   <xacro:base_v0 parent="base_footprint">
 	<origin xyz="0 0 0" rpy="0 0 ${-M_PI/2}"/>
-	<origin xyz="0 0 0" rpy="0 0 0"/>
+	<origin xyz="0 0 0.369" rpy="0 0 0"/>
   </xacro:base_v0>
   <!-- Rocker -->
@@ -35,5 +35,5 @@
   			 iyy="0.002" iyz="-0.0000001149"
   			 izz="0.003"/>
-  	<origin xyz="0.2 -0.02 -0.15" rpy="0 0 ${M_PI}"/>
+  	<origin xyz="0.2 -0.019945 -0.15" rpy="0 0 ${M_PI}"/>
   	<axis xyz="0 1 0"/>
   </xacro:bogie_v0>
@@ -43,5 +43,5 @@
   			 iyy="0.002" iyz="0.0000001156"
   			 izz="0.003"/>
-  	<origin xyz="0.21 0.02 -0.14" rpy="0 0 ${M_PI}"/>
+  	<origin xyz="0.2 0.019945 -0.15" rpy="0 0 ${M_PI}"/>
   	<axis xyz="0 1 0"/>
   </xacro:bogie_v0>
@@ -49,52 +49,52 @@
   <xacro:support_v0 part="right_front" parent="bogie_right_link">
   	<origin xyz="0 0 0" rpy="0 0 0"/>
-  	<origin xyz="-0.202 0.1475 -0.175" rpy="0 0 ${-M_PI/2}"/>
+  	<origin xyz="-0.202 0.115 0.05" rpy="0 0 ${-M_PI/2}"/>
   	<axis xyz="0 0 1"/>
   </xacro:support_v0>
-  <!-- <xacro:support_v0 part="right_back" parent="rocker_right_link"> -->
-  <!-- 	<origin xyz="0 0 0" rpy="0 0 0"/> -->
-  <!-- 	<origin xyz="0 0 0" rpy="0 0 0"/> -->
-  <!-- 	<axis xyz="1 0 0"/> -->
-  <!-- </xacro:support_v0> -->
-  <!-- <xacro:support_v0 part="left_front" parent="bogie_left_link"> -->
-  <!-- 	<origin xyz="0 0 0" rpy="0 0 0"/> -->
-  <!-- 	<origin xyz="0 0 0" rpy="0 0 0"/> -->
-  <!-- 	<axis xyz="1 0 0"/> -->
-  <!-- </xacro:support_v0> -->
-  <!-- <xacro:support_v0 part="left_back" parent="rocker_left_link"> -->
-  <!-- 	<origin xyz="0 0 0" rpy="0 0 0"/> -->
-  <!-- 	<origin xyz="0 0 0" rpy="0 0 0"/> -->
-  <!-- 	<axis xyz="1 0 0"/> -->
-  <!-- </xacro:support_v0> -->
+  <xacro:support_v0 part="right_back" parent="rocker_right_link">
+  	<origin xyz="0 0 0" rpy="0 0 0"/>
+  	<origin xyz="-0.4 -0.05 -0.1" rpy="0 0 ${M_PI/2}"/>
+  	<axis xyz="0 0 1"/>
+  </xacro:support_v0>
+  <xacro:support_v0 part="left_front" parent="bogie_left_link">
+  	<origin xyz="0 0 0" rpy="0 0 0"/>
+  	<origin xyz="-0.202 -0.115 0.05" rpy="0 0 ${M_PI/2}"/>
+  	<axis xyz="0 0 1"/>
+  </xacro:support_v0>
+  <xacro:support_v0 part="left_back" parent="rocker_left_link">
+  	<origin xyz="0 0 0" rpy="0 0 0"/>
+  	<origin xyz="-0.4 0.05 -0.1" rpy="0 0 ${-M_PI/2}"/>
+  	<axis xyz="0 0 1"/>
+  </xacro:support_v0>
   <!-- Wheel -->
-  <!-- <xacro:wheel_v0 part="right_front" parent="support_right_front_link"> -->
-  <!-- 	<origin xyz="0 0 0" rpy="0 0 0"/> -->
-  <!-- 	<oritin xyz="0 0 0" rpy="0 0 0"/> -->
-  <!-- 	<axis xyz="1 0 0"/> -->
-  <!-- </xacro:wheel_v0> -->
-  <!-- <xacro:wheel_v0 part="right_middle" parent="bogie_right_link"> -->
-  <!-- 	<origin xyz="0 0 0" rpy="0 0 0"/> -->
-  <!-- 	<oritin xyz="0 0 0" rpy="0 0 0"/> -->
-  <!-- 	<axis xyz="1 0 0"/> -->
-  <!-- </xacro:wheel_v0> -->
-  <!-- <xacro:wheel_v0 part="right_back" parent="support_right_back_link"> -->
-  <!-- 	<origin xyz="0 0 0" rpy="0 0 0"/> -->
-  <!-- 	<oritin xyz="0 0 0" rpy="0 0 0"/> -->
-  <!-- 	<axis xyz="1 0 0"/> -->
-  <!-- </xacro:wheel_v0> -->
-  <!-- <xacro:wheel_v0 part="left_front" parent="support_left_front_link"> -->
-  <!-- 	<origin xyz="0 0 0" rpy="0 0 0"/> -->
-  <!-- 	<oritin xyz="0 0 0" rpy="0 0 0"/> -->
-  <!-- 	<axis xyz="1 0 0"/> -->
-  <!-- </xacro:wheel_v0> -->
-  <!-- <xacro:wheel_v0 part="left_middle" parent="bogie_left_link"> -->
-  <!-- 	<origin xyz="0 0 0" rpy="0 0 0"/> -->
-  <!-- 	<oritin xyz="0 0 0" rpy="0 0 0"/> -->
-  <!-- 	<axis xyz="1 0 0"/> -->
-  <!-- </xacro:wheel_v0> -->
-  <!-- <xacro:wheel_v0 part="left_back" parent="support_left_back_link"> -->
-  <!-- 	<origin xyz="0 0 0" rpy="0 0 0"/> -->
-  <!-- 	<oritin xyz="0 0 0" rpy="0 0 0"/> -->
-  <!-- 	<axis xyz="1 0 0"/> -->
-  <!-- </xacro:wheel_v0> -->
+  <xacro:wheel_v0 part="right_front" parent="support_right_front_link">
+  	<origin xyz="0 0 0" rpy="0 0 0"/>
+  	<origin xyz="-0.065 0 -0.2145" rpy="0 0 0"/>
+  	<axis xyz="1 0 0"/>
+  </xacro:wheel_v0>
+  <xacro:wheel_v0 part="right_middle" parent="bogie_right_link">
+  	<origin xyz="0 0 0" rpy="0 0 0"/>
+  	<origin xyz="0.198 0.2485 -0.165" rpy="0 0 ${-M_PI/2}"/>
+  	<axis xyz="1 0 0"/>
+  </xacro:wheel_v0>
+  <xacro:wheel_v0 part="right_back" parent="support_right_back_link">
+  	<origin xyz="0 0 0" rpy="0 0 0"/>
+  	<origin xyz="-0.065 0 -0.2145" rpy="0 0 0"/>
+  	<axis xyz="1 0 0"/>
+  </xacro:wheel_v0>
+  <xacro:wheel_v0 part="left_front" parent="support_left_front_link">
+  	<origin xyz="0 0 0" rpy="0 0 0"/>
+  	<origin xyz="-0.065 0 -0.2145" rpy="0 0 0"/>
+  	<axis xyz="1 0 0"/>
+  </xacro:wheel_v0>
+  <xacro:wheel_v0 part="left_middle" parent="bogie_left_link">
+  	<origin xyz="0 0 0" rpy="0 0 0"/>
+  	<origin xyz="0.198 -0.2485 -0.165" rpy="0 0 ${M_PI/2}"/>
+  	<axis xyz="1 0 0"/>
+  </xacro:wheel_v0>
+  <xacro:wheel_v0 part="left_back" parent="support_left_back_link">
+  	<origin xyz="0 0 0" rpy="0 0 0"/>
+  	<origin xyz="-0.065 0 -0.2145" rpy="0 0 0"/>
+  	<axis xyz="1 0 0"/>
+  </xacro:wheel_v0>
 </robot>

File: fr01_description/urdf/wheel/wheel.urdf.xacro (robot description, xacro)
@@ -52,7 +52,7 @@
       </collision>
       <inertial>
-        <mass value="2.517"/>
-        <inertia ixx="0.0005746" ixy="0.0000000001176" ixz="0.0000003448"
-				 iyy="0.002" iyz="-0.0000000007211"
+        <mass value="2.522"/>
+        <inertia ixx="0.0005737" ixy="0.0000000001174" ixz="0.0000003442"
+				 iyy="0.002" iyz="-0.0000000007199"
 				 izz="0.002" />
       </inertial>

Commit message: [rename] rename support_link to steer_link

File: fr01_description/robots/fr01.urdf.xacro (robot description, xacro)
@@ -47,27 +47,27 @@
   	<axis xyz="0 1 0"/>
   </xacro:bogie_v0>
-  <!-- Support -->
-  <xacro:support_v0 part="right_front" parent="bogie_right_link">
+  <!-- Steer -->
+  <xacro:steer_v0 part="right_front" parent="bogie_right_link">
   	<origin xyz="0 0 0" rpy="0 0 0"/>
   	<origin xyz="-0.202 0.115 0.05" rpy="0 0 ${-M_PI/2}"/>
   	<axis xyz="0 0 1"/>
-  </xacro:support_v0>
-  <xacro:support_v0 part="right_back" parent="rocker_right_link">
+  </xacro:steer_v0>
+  <xacro:steer_v0 part="right_back" parent="rocker_right_link">
   	<origin xyz="0 0 0" rpy="0 0 0"/>
   	<origin xyz="-0.4 -0.05 -0.1" rpy="0 0 ${M_PI/2}"/>
   	<axis xyz="0 0 1"/>
-  </xacro:support_v0>
-  <xacro:support_v0 part="left_front" parent="bogie_left_link">
+  </xacro:steer_v0>
+  <xacro:steer_v0 part="left_front" parent="bogie_left_link">
   	<origin xyz="0 0 0" rpy="0 0 0"/>
   	<origin xyz="-0.202 -0.115 0.05" rpy="0 0 ${M_PI/2}"/>
   	<axis xyz="0 0 1"/>
-  </xacro:support_v0>
-  <xacro:support_v0 part="left_back" parent="rocker_left_link">
+  </xacro:steer_v0>
+  <xacro:steer_v0 part="left_back" parent="rocker_left_link">
   	<origin xyz="0 0 0" rpy="0 0 0"/>
   	<origin xyz="-0.4 0.05 -0.1" rpy="0 0 ${-M_PI/2}"/>
   	<axis xyz="0 0 1"/>
-  </xacro:support_v0>
+  </xacro:steer_v0>
   <!-- Wheel -->
-  <xacro:wheel_v0 part="right_front" parent="support_right_front_link">
+  <xacro:wheel_v0 part="right_front" parent="steer_right_front_link">
   	<origin xyz="0 0 0" rpy="0 0 0"/>
   	<origin xyz="-0.065 0 -0.2145" rpy="0 0 0"/>
@@ -79,10 +79,10 @@
   	<axis xyz="1 0 0"/>
   </xacro:wheel_v0>
-  <xacro:wheel_v0 part="right_back" parent="support_right_back_link">
+  <xacro:wheel_v0 part="right_back" parent="steer_right_back_link">
   	<origin xyz="0 0 0" rpy="0 0 0"/>
   	<origin xyz="-0.065 0 -0.2145" rpy="0 0 0"/>
   	<axis xyz="1 0 0"/>
   </xacro:wheel_v0>
-  <xacro:wheel_v0 part="left_front" parent="support_left_front_link">
+  <xacro:wheel_v0 part="left_front" parent="steer_left_front_link">
   	<origin xyz="0 0 0" rpy="0 0 0"/>
   	<origin xyz="-0.065 0 -0.2145" rpy="0 0 0"/>
@@ -94,5 +94,5 @@
   	<axis xyz="1 0 0"/>
   </xacro:wheel_v0>
-  <xacro:wheel_v0 part="left_back" parent="support_left_back_link">
+  <xacro:wheel_v0 part="left_back" parent="steer_left_back_link">
   	<origin xyz="0 0 0" rpy="0 0 0"/>
   	<origin xyz="-0.065 0 -0.2145" rpy="0 0 0"/>
@@ -106,9 +106,9 @@
   <xacro:bogie_trans_v0 side="right"/>
   <xacro:bogie_trans_v0 side="left"/>
-  <!-- Support -->
-  <xacro:support_trans_v0 part="right_front"/>
-  <xacro:support_trans_v0 part="right_back"/>
-  <xacro:support_trans_v0 part="left_front"/>
-  <xacro:support_trans_v0 part="left_back"/>
+  <!-- Steer -->
+  <xacro:steer_trans_v0 part="right_front"/>
+  <xacro:steer_trans_v0 part="right_back"/>
+  <xacro:steer_trans_v0 part="left_front"/>
+  <xacro:steer_trans_v0 part="left_back"/>
   <!-- Wheel -->
   <xacro:wheel_trans_v0 part="right_front"/>
@@ -127,9 +127,9 @@
   <xacro:bogie_gazebo_v0 side="right"/>
   <xacro:bogie_gazebo_v0 side="left"/>
-  <!-- Support -->
-  <xacro:support_gazebo_v0 part="right_front"/>
-  <xacro:support_gazebo_v0 part="right_back"/>
-  <xacro:support_gazebo_v0 part="left_front"/>
-  <xacro:support_gazebo_v0 part="left_back"/>
+  <!-- Steer -->
+  <xacro:steer_gazebo_v0 part="right_front"/>
+  <xacro:steer_gazebo_v0 part="right_back"/>
+  <xacro:steer_gazebo_v0 part="left_front"/>
+  <xacro:steer_gazebo_v0 part="left_back"/>
   <!-- Wheel -->
   <xacro:wheel_gazebo_v0 part="right_front"/>

File: fr01_description/urdf/wheel/wheel.gazebo.xacro (robot description, xacro)
@@ -8,5 +8,5 @@
     </gazebo>
   </xacro:macro>
-  <xacro:macro name="support_gazebo_v0" params="part">
+  <xacro:macro name="steer_gazebo_v0" params="part">
 	<gazebo reference="rocke_${part}_link">
 	  <selfCollide>true</selfCollide>

File: fr01_description/urdf/wheel/wheel.transmission.xacro (robot description, xacro)
@@ -13,11 +13,11 @@
 	</transmission>
   </xacro:macro>
-  <xacro:macro name="support_trans_v0" params="part">
-	<transmission name="support_${part}_trans">
+  <xacro:macro name="steer_trans_v0" params="part">
+	<transmission name="steer_${part}_trans">
       <type>transmission_interface/SimpleTransmission</type>
-      <joint name="support_${part}_joint">
+      <joint name="steer_${part}_joint">
 		<hardwareInterface>EffortJointInterface</hardwareInterface>
       </joint>
-	  <actuator name="support_${part}_motor">
+	  <actuator name="steer_${part}_motor">
 		<hardwareInterface>EffortJointInterface</hardwareInterface>
 		<mechanicalReduction>1</mechanicalReduction>

File: fr01_description/urdf/wheel/wheel.urdf.xacro (robot description, xacro)
@@ -31,18 +31,18 @@
     </link>
   </xacro:macro>
-  <xacro:macro name="support_v0" params="part parent *link_origin *joint_origin *joint_axis">
-	<joint name="support_${part}_joint" type="revolute">
+  <xacro:macro name="steer_v0" params="part parent *link_origin *joint_origin *joint_axis">
+	<joint name="steer_${part}_joint" type="revolute">
 	  <insert_block name="joint_origin"/>
 	  <parent link="${parent}"/>
-	  <child link="support_${part}_link"/>
+	  <child link="steer_${part}_link"/>
 	  <insert_block name="joint_axis"/>
 	  <dynamics dampint="0.7" friction="0.7"/>
 	  <limit effort="30.0" lower="${-M_PI/2}" upper="${M_PI/2}" velocity="${2*M_PI}"/>
 	</joint>
-    <link name="support_${part}_link">
+    <link name="steer_${part}_link">
       <visual>
 		<insert_block name="link_origin"/>
         <geometry>
-          <mesh filename="package://fr01_description/meshes/visual/support_link.dae"/>
+          <mesh filename="package://fr01_description/meshes/visual/steer_link.dae"/>
         </geometry>
       </visual>
@@ -50,5 +50,5 @@
 		<insert_block name="link_origin"/>
         <geometry>
-		  <mesh filename="package://fr01_description/meshes/collision/support_link.stl"/>
+		  <mesh filename="package://fr01_description/meshes/collision/steer_link.stl"/>
         </geometry>
       </collision>

Commit message: [modify] modify the base_footprint height
modify the height from base_footprint to base_link

File: fr01_description/robots/fr01.urdf.xacro (robot description, xacro)
@@ -11,5 +11,5 @@
   <xacro:base_v0 parent="base_footprint">
 	<origin xyz="0 0 0" rpy="0 0 ${-M_PI/2}"/>
-	<origin xyz="0 0 0.369" rpy="0 0 0"/>
+	<origin xyz="0 0 0.370" rpy="0 0 0"/>
   </xacro:base_v0>
   <!-- Rocker -->

File: fr01_description/robots/urdf/fr01.urdf (robot description, URDF)
Before this commit: robot fr01, 16 links, 15 joints
Joints:
- joint base_link_joint: origin xyz=0 0 0.369 rpy=0 0 0 -> xyz=0 0 0.370 rpy=0 0 0

Commit message: [modify] modify base_footprint
On this robot, the base_link frame will move.
So, If we want base_footprint frame(always on grand surface),
we need to change the parent-child relationship.
That is the parent of base_footprint is rocker_right_link.

File: fr01_description/robots/fr01.urdf.xacro (robot description, xacro)
@@ -8,6 +8,6 @@
   <!--==================== Link & Joint ====================-->
   <!-- Body -->
-  <link name="base_footprint"/>
-  <xacro:base_v0 parent="base_footprint">
+  <link name="fake_base_footprint"/>
+  <xacro:base_v0 parent="fake_base_footprint">
 	<origin xyz="0 0 0" rpy="0 0 ${-M_PI/2}"/>
 	<origin xyz="0 0 0.370" rpy="0 0 0"/>
@@ -99,4 +99,10 @@
   	<axis xyz="1 0 0"/>
   </xacro:wheel_v0>
+  <link name="base_footprint"/>
+  <joint name="base_footprint_joint" type="fixed">
+	<origin xyz="0 0.213 -0.398" rpy="0 0 0"/>
+	<parent link="rocker_right_link"/>
+	<child link="base_footprint"/>
+  </joint>
   <!--==================== Transmission ====================-->
   <!-- Rocker -->
@@ -119,4 +125,9 @@
   <xacro:wheel_trans_v0 part="left_back"/>
   <!--==================== Gazebo ====================-->
+  <gazebo>
+    <plugin name="gazebo_ros_control" filename="libgazebo_ros_control.so">
+      <robotNamespace>/fr01</robotNamespace>
+    </plugin>
+  </gazebo>
   <!-- Body -->
   <xacro:body_gazebo_vo/>

File: fr01_description/robots/urdf/fr01.urdf (robot description, URDF)
Before this commit: robot fr01, 16 links, 15 joints
Links:
- added link fake_base_footprint
Joints:
- added joint base_footprint_joint: type fixed, parent rocker_right_link, child base_footprint, origin xyz=0 0.213 -0.398 rpy=0 0 0
- joint base_link_joint: parent base_footprint -> fake_base_footprint

Commit message: [modify] apply diff_drive_controller

File: fr01_description/robots/fr01.urdf.xacro (robot description, xacro)
@@ -125,7 +125,20 @@
   <xacro:wheel_trans_v0 part="left_back"/>
   <!--==================== Gazebo ====================-->
+  <!-- firstly load diff_drive_controller without namespaces -->
   <gazebo>
     <plugin name="gazebo_ros_control" filename="libgazebo_ros_control.so">
-      <robotNamespace>/fr01</robotNamespace>
+    </plugin>
+  </gazebo>
+  <!-- Wheel -->
+  <xacro:wheel_gazebo_v0 part="right_front"/>
+  <xacro:wheel_gazebo_v0 part="right_middle"/>
+  <xacro:wheel_gazebo_v0 part="right_back"/>
+  <xacro:wheel_gazebo_v0 part="left_front"/>
+  <xacro:wheel_gazebo_v0 part="left_middle"/>
+  <xacro:wheel_gazebo_v0 part="left_back"/>
+  <!-- secondly load other controllers with namespace -->
+  <gazebo>
+    <plugin name="gazebo_ros_control" filename="libgazebo_ros_control.so">
+        <robotNamespace>/fr01</robotNamespace>
     </plugin>
   </gazebo>
@@ -143,10 +156,3 @@
   <xacro:steer_gazebo_v0 part="left_front"/>
   <xacro:steer_gazebo_v0 part="left_back"/>
-  <!-- Wheel -->
-  <xacro:wheel_gazebo_v0 part="right_front"/>
-  <xacro:wheel_gazebo_v0 part="right_middle"/>
-  <xacro:wheel_gazebo_v0 part="right_back"/>
-  <xacro:wheel_gazebo_v0 part="left_front"/>
-  <xacro:wheel_gazebo_v0 part="left_middle"/>
-  <xacro:wheel_gazebo_v0 part="left_back"/>
 </robot>

File: fr01_description/urdf/wheel/wheel.transmission.xacro (robot description, xacro)
@@ -1,27 +1,27 @@
 <?xml version="1.0"?>
 <robot xmlns:xacro="http://ros.org/wiki/xacro">
-  <xacro:macro name="wheel_trans_v0" params="part">
-	<transmission name="wheel_${part}_trans">
-      <type>transmission_interface/SimpleTransmission</type>
-      <joint name="wheel_${part}_joint">
-		<hardwareInterface>EffortJointInterface</hardwareInterface>
-      </joint>
-	  <actuator name="wheel_${part}_motor">
-		<hardwareInterface>EffortJointInterface</hardwareInterface>
-		<mechanicalReduction>50</mechanicalReduction>
-      </actuator>
-	</transmission>
-  </xacro:macro>
-  <xacro:macro name="steer_trans_v0" params="part">
-	<transmission name="steer_${part}_trans">
-      <type>transmission_interface/SimpleTransmission</type>
-      <joint name="steer_${part}_joint">
-		<hardwareInterface>EffortJointInterface</hardwareInterface>
-      </joint>
-	  <actuator name="steer_${part}_motor">
-		<hardwareInterface>EffortJointInterface</hardwareInterface>
-		<mechanicalReduction>1</mechanicalReduction>
-      </actuator>
-	</transmission>
-  </xacro:macro>
+    <xacro:macro name="wheel_trans_v0" params="part">
+        <transmission name="wheel_${part}_trans">
+            <type>transmission_interface/SimpleTransmission</type>
+            <joint name="wheel_${part}_joint">
+                <hardwareInterface>VelocityJointInterface</hardwareInterface>
+            </joint>
+            <actuator name="wheel_${part}_motor">
+                <hardwareInterface>VelocityJointInterface</hardwareInterface>
+                <mechanicalReduction>50</mechanicalReduction>
+            </actuator>
+        </transmission>
+    </xacro:macro>
+    <xacro:macro name="steer_trans_v0" params="part">
+        <transmission name="steer_${part}_trans">
+            <type>transmission_interface/SimpleTransmission</type>
+            <joint name="steer_${part}_joint">
+                <hardwareInterface>PositionJointInterface</hardwareInterface>
+            </joint>
+            <actuator name="steer_${part}_motor">
+                <hardwareInterface>PositionJointInterface</hardwareInterface>
+                <mechanicalReduction>1</mechanicalReduction>
+            </actuator>
+        </transmission>
+    </xacro:macro>
 </robot>

File: fr01_description/urdf/wheel/wheel.urdf.xacro (robot description, xacro)
@@ -3,4 +3,6 @@
   <xacro:include filename="$(find fr01_description)/urdf/wheel/wheel.transmission.xacro"/>
   <xacro:include filename="$(find fr01_description)/urdf/wheel/wheel.gazebo.xacro"/>
+  <xacro:property name="wheel_radius" value="0.03"/>
+  <xacro:property name="wheel_width" value="0.02"/>
   <xacro:macro name="wheel_v0" params="part parent *link_origin *joint_origin *joint_axis">
 	<joint name="wheel_${part}_joint" type="continuous">
@@ -20,5 +22,6 @@
 		<insert_block name="link_origin"/>
         <geometry>
-		  <mesh filename="package://fr01_description/meshes/collision/wheel_link.stl"/>
+            <!-- <mesh filename="package://fr01_description/meshes/collision/wheel_link.stl"/> -->
+            <cylinder radius="${wheel_radius}" length="${wheel_width}"/>
         </geometry>
       </collision>

Commit message: [WIP] removed namespace to activate diff_drive_controller

File: fr01_description/robots/fr01.urdf.xacro (robot description, xacro)
@@ -137,18 +137,16 @@
   <xacro:wheel_gazebo_v0 part="left_middle"/>
   <xacro:wheel_gazebo_v0 part="left_back"/>
-  <!-- secondly load other controllers with namespace -->
-  <gazebo>
-    <plugin name="gazebo_ros_control" filename="libgazebo_ros_control.so">
-        <robotNamespace>/fr01</robotNamespace>
-    </plugin>
-  </gazebo>
   <!-- Body -->
   <xacro:body_gazebo_vo/>
   <!-- Rocker -->
+<!--
   <xacro:rocker_gazebo_v0 side="right"/>
   <xacro:rocker_gazebo_v0 side="left"/>
+-->
   <!-- Bogie -->
+<!--
   <xacro:bogie_gazebo_v0 side="right"/>
   <xacro:bogie_gazebo_v0 side="left"/>
+-->
   <!-- Steer -->
   <xacro:steer_gazebo_v0 part="right_front"/>

File: fr01_description/urdf/leg/leg.urdf.xacro (robot description, xacro)
@@ -9,5 +9,5 @@
 	  <child link="bogie_${side}_link"/>
 	  <insert_block name="joint_axis"/>
-	  <dynamics dampint="0.7" friction="0.7"/>
+	  <dynamics dampint="0.04" friction="0.01"/>
 	  <limit effort="30.0" lower="${-M_PI/2}" upper="${M_PI/2}" velocity="${2*M_PI}"/>
 	</joint>
@@ -37,5 +37,5 @@
 	  <child link="rocker_${side}_link"/>
 	  <insert_block name="joint_axis"/>
-	  <dynamics dampint="0.7" friction="0.7"/>
+	  <dynamics dampint="1.4" friction="1.0"/>
 	  <limit effort="30.0" lower="${-M_PI/2}" upper="${M_PI/2}" velocity="${2*M_PI}"/>
 	</joint>

File: fr01_description/urdf/wheel/wheel.urdf.xacro (robot description, xacro)
@@ -3,6 +3,6 @@
   <xacro:include filename="$(find fr01_description)/urdf/wheel/wheel.transmission.xacro"/>
   <xacro:include filename="$(find fr01_description)/urdf/wheel/wheel.gazebo.xacro"/>
-  <xacro:property name="wheel_radius" value="0.03"/>
-  <xacro:property name="wheel_width" value="0.02"/>
+  <xacro:property name="wheel_radius" value="0.08"/>
+  <xacro:property name="wheel_width" value="0.16"/>
   <xacro:macro name="wheel_v0" params="part parent *link_origin *joint_origin *joint_axis">
 	<joint name="wheel_${part}_joint" type="continuous">
@@ -20,6 +20,7 @@
       </visual>
       <collision>
-		<insert_block name="link_origin"/>
-        <geometry>
+          <!-- <insert_block name="link_origin"/> -->
+          <origin xyz="0 0 0" rpy="0 ${M_PI/2} 0"/>
+          <geometry>
             <!-- <mesh filename="package://fr01_description/meshes/collision/wheel_link.stl"/> -->
             <cylinder radius="${wheel_radius}" length="${wheel_width}"/>
