Commit message: [fix] fixed joint configuration for diff_drive_controller

File: fr01_description/robots/fr01.urdf.xacro (robot description, xacro)
@@ -73,4 +73,5 @@
   	<origin xyz="-0.065 0 -0.2145" rpy="0 0 0"/>
   	<axis xyz="1 0 0"/>
+  	<origin xyz="0.065 0 0" rpy="0 ${M_PI/2} 0"/>
   </xacro:wheel_v0>
   <xacro:wheel_v0 part="right_middle" parent="bogie_right_link">
@@ -78,4 +79,5 @@
   	<origin xyz="0.198 0.2485 -0.165" rpy="0 0 ${-M_PI/2}"/>
   	<axis xyz="1 0 0"/>
+  	<origin xyz="0.065 0 0" rpy="0 ${M_PI/2} 0"/>
   </xacro:wheel_v0>
   <xacro:wheel_v0 part="right_back" parent="steer_right_back_link">
@@ -83,19 +85,23 @@
   	<origin xyz="-0.065 0 -0.2145" rpy="0 0 0"/>
   	<axis xyz="1 0 0"/>
+  	<origin xyz="0.065 0 0" rpy="0 ${M_PI/2} 0"/>
   </xacro:wheel_v0>
   <xacro:wheel_v0 part="left_front" parent="steer_left_front_link">
-  	<origin xyz="0 0 0" rpy="0 0 0"/>
-  	<origin xyz="-0.065 0 -0.2145" rpy="0 0 0"/>
+  	<origin xyz="0 0 0" rpy="0 ${M_PI} 0"/>
+  	<origin xyz="-0.065 0 -0.2145" rpy="0 ${M_PI} 0"/>
   	<axis xyz="1 0 0"/>
+  	<origin xyz="-0.065 0 0" rpy="0 ${M_PI/2} 0"/>
   </xacro:wheel_v0>
   <xacro:wheel_v0 part="left_middle" parent="bogie_left_link">
-  	<origin xyz="0 0 0" rpy="0 0 0"/>
-  	<origin xyz="0.198 -0.2485 -0.165" rpy="0 0 ${M_PI/2}"/>
+  	<origin xyz="0 0 0" rpy="0 ${M_PI} 0"/>
+  	<origin xyz="0.198 -0.2485 -0.165" rpy="0 ${M_PI} ${M_PI/2}"/>
   	<axis xyz="1 0 0"/>
+  	<origin xyz="-0.065 0 0" rpy="0 ${M_PI/2} 0"/>
   </xacro:wheel_v0>
   <xacro:wheel_v0 part="left_back" parent="steer_left_back_link">
-  	<origin xyz="0 0 0" rpy="0 0 0"/>
-  	<origin xyz="-0.065 0 -0.2145" rpy="0 0 0"/>
+  	<origin xyz="0 0 0" rpy="0 ${M_PI} 0"/>
+  	<origin xyz="-0.065 0 -0.2145" rpy="0 ${M_PI} 0"/>
   	<axis xyz="1 0 0"/>
+  	<origin xyz="-0.065 0 0" rpy="0 ${M_PI/2} 0"/>
   </xacro:wheel_v0>
   <link name="base_footprint"/>
@@ -140,13 +146,9 @@
   <xacro:body_gazebo_vo/>
   <!-- Rocker -->
-<!--
   <xacro:rocker_gazebo_v0 side="right"/>
   <xacro:rocker_gazebo_v0 side="left"/>
--->
   <!-- Bogie -->
-<!--
   <xacro:bogie_gazebo_v0 side="right"/>
   <xacro:bogie_gazebo_v0 side="left"/>
--->
   <!-- Steer -->
   <xacro:steer_gazebo_v0 part="right_front"/>

File: fr01_description/urdf/wheel/wheel.urdf.xacro (robot description, xacro)
@@ -5,5 +5,5 @@
   <xacro:property name="wheel_radius" value="0.08"/>
   <xacro:property name="wheel_width" value="0.16"/>
-  <xacro:macro name="wheel_v0" params="part parent *link_origin *joint_origin *joint_axis">
+  <xacro:macro name="wheel_v0" params="part parent *link_origin *joint_origin *joint_axis *collision_origin">
 	<joint name="wheel_${part}_joint" type="continuous">
 	  <insert_block name="joint_origin"/>
@@ -20,8 +20,8 @@
       </visual>
       <collision>
-          <!-- <insert_block name="link_origin"/> -->
-          <origin xyz="0 0 0" rpy="0 ${M_PI/2} 0"/>
+          <insert_block name="collision_origin"/>
           <geometry>
             <!-- <mesh filename="package://fr01_description/meshes/collision/wheel_link.stl"/> -->
+            <!-- diff drive controller assumese the collision is cylinder -->
             <cylinder radius="${wheel_radius}" length="${wheel_width}"/>
         </geometry>

Commit message: [modify] replace wheel params with xacro property

File: fr01_description/robots/fr01.urdf.xacro (robot description, xacro)
@@ -6,4 +6,7 @@
   <xacro:include filename="$(find fr01_description)/urdf/leg/leg.urdf.xacro"/>
   <xacro:include filename="$(find fr01_description)/urdf/wheel/wheel.urdf.xacro"/>
+  <!-- wheel parameters -->
+  <xacro:property name="wheel_radius" value="0.08"/>
+  <xacro:property name="wheel_width" value="0.16"/>
   <!--==================== Link & Joint ====================-->
   <!-- Body -->
@@ -69,5 +72,6 @@
   </xacro:steer_v0>
   <!-- Wheel -->
-  <xacro:wheel_v0 part="right_front" parent="steer_right_front_link">
+  <xacro:wheel_v0 part="right_front" parent="steer_right_front_link"
+      wheel_radius="${wheel_radius}" wheel_width="${wheel_width}">
   	<origin xyz="0 0 0" rpy="0 0 0"/>
   	<origin xyz="-0.065 0 -0.2145" rpy="0 0 0"/>
@@ -75,5 +79,6 @@
   	<origin xyz="0.065 0 0" rpy="0 ${M_PI/2} 0"/>
   </xacro:wheel_v0>
-  <xacro:wheel_v0 part="right_middle" parent="bogie_right_link">
+  <xacro:wheel_v0 part="right_middle" parent="bogie_right_link"
+      wheel_radius="${wheel_radius}" wheel_width="${wheel_width}">
   	<origin xyz="0 0 0" rpy="0 0 0"/>
   	<origin xyz="0.198 0.2485 -0.165" rpy="0 0 ${-M_PI/2}"/>
@@ -81,5 +86,6 @@
   	<origin xyz="0.065 0 0" rpy="0 ${M_PI/2} 0"/>
   </xacro:wheel_v0>
-  <xacro:wheel_v0 part="right_back" parent="steer_right_back_link">
+  <xacro:wheel_v0 part="right_back" parent="steer_right_back_link"
+      wheel_radius="${wheel_radius}" wheel_width="${wheel_width}">
   	<origin xyz="0 0 0" rpy="0 0 0"/>
   	<origin xyz="-0.065 0 -0.2145" rpy="0 0 0"/>
@@ -87,5 +93,6 @@
   	<origin xyz="0.065 0 0" rpy="0 ${M_PI/2} 0"/>
   </xacro:wheel_v0>
-  <xacro:wheel_v0 part="left_front" parent="steer_left_front_link">
+  <xacro:wheel_v0 part="left_front" parent="steer_left_front_link"
+      wheel_radius="${wheel_radius}" wheel_width="${wheel_width}">
   	<origin xyz="0 0 0" rpy="0 ${M_PI} 0"/>
   	<origin xyz="-0.065 0 -0.2145" rpy="0 ${M_PI} 0"/>
@@ -93,5 +100,6 @@
   	<origin xyz="-0.065 0 0" rpy="0 ${M_PI/2} 0"/>
   </xacro:wheel_v0>
-  <xacro:wheel_v0 part="left_middle" parent="bogie_left_link">
+  <xacro:wheel_v0 part="left_middle" parent="bogie_left_link"
+      wheel_radius="${wheel_radius}" wheel_width="${wheel_width}">
   	<origin xyz="0 0 0" rpy="0 ${M_PI} 0"/>
   	<origin xyz="0.198 -0.2485 -0.165" rpy="0 ${M_PI} ${M_PI/2}"/>
@@ -99,5 +107,6 @@
   	<origin xyz="-0.065 0 0" rpy="0 ${M_PI/2} 0"/>
   </xacro:wheel_v0>
-  <xacro:wheel_v0 part="left_back" parent="steer_left_back_link">
+  <xacro:wheel_v0 part="left_back" parent="steer_left_back_link"
+      wheel_radius="${wheel_radius}" wheel_width="${wheel_width}">
   	<origin xyz="0 0 0" rpy="0 ${M_PI} 0"/>
   	<origin xyz="-0.065 0 -0.2145" rpy="0 ${M_PI} 0"/>

File: fr01_description/urdf/wheel/wheel.urdf.xacro (robot description, xacro)
@@ -3,7 +3,6 @@
   <xacro:include filename="$(find fr01_description)/urdf/wheel/wheel.transmission.xacro"/>
   <xacro:include filename="$(find fr01_description)/urdf/wheel/wheel.gazebo.xacro"/>
-  <xacro:property name="wheel_radius" value="0.08"/>
-  <xacro:property name="wheel_width" value="0.16"/>
-  <xacro:macro name="wheel_v0" params="part parent *link_origin *joint_origin *joint_axis *collision_origin">
+  <xacro:macro name="wheel_v0" params="part parent wheel_radius wheel_width
+      *link_origin *joint_origin *joint_axis *collision_origin">
 	<joint name="wheel_${part}_joint" type="continuous">
 	  <insert_block name="joint_origin"/>

Commit message: [modify] add stabilized_base_link
Added but it not works....omg

File: fr01_description/robots/fr01.urdf.xacro (robot description, xacro)
@@ -10,9 +10,15 @@
   <xacro:property name="wheel_width" value="0.16"/>
   <!--==================== Link & Joint ====================-->
+  <link name="base_footprint"/>
+  <joint name="base_footprint_joint" type="fixed">
+	<origin xyz="0 0 0.370" rpy="0 0 0"/>
+	<parent link="base_footprint"/>
+	<child link="stabilized_base_link"/>
+  </joint>
   <!-- Body -->
-  <link name="fake_base_footprint"/>
-  <xacro:base_v0 parent="fake_base_footprint">
+  <link name="stabilized_base_link"/>
+  <xacro:base_v0 parent="stabilized_base_link">
 	<origin xyz="0 0 0" rpy="0 0 ${-M_PI/2}"/>
-	<origin xyz="0 0 0.370" rpy="0 0 0"/>
+	<origin xyz="0 0 0" rpy="0 0 0"/>
   </xacro:base_v0>
   <!-- Rocker -->
@@ -114,10 +120,4 @@
   	<origin xyz="-0.065 0 0" rpy="0 ${M_PI/2} 0"/>
   </xacro:wheel_v0>
-  <link name="base_footprint"/>
-  <joint name="base_footprint_joint" type="fixed">
-	<origin xyz="0 0.213 -0.398" rpy="0 0 0"/>
-	<parent link="rocker_right_link"/>
-	<child link="base_footprint"/>
-  </joint>
   <!--==================== Transmission ====================-->
   <!-- Rocker -->

File: fr01_description/urdf/body/body.urdf.xacro (robot description, xacro)
@@ -3,8 +3,9 @@
   <xacro:include filename="$(find fr01_description)/urdf/body/body.gazebo.xacro"/>
   <xacro:macro name="base_v0" params="parent *link_origin *joint_origin">
-	<joint name="base_link_joint" type="fixed">
+	<joint name="base_link_joint" type="continuous">
       <insert_block name="joint_origin" />
       <parent link="${parent}"/>
       <child link="base_link"/>
+	  <axis xyz="1 1 0"/>
 	</joint>
     <link name="base_link">

Commit message: [modify] add base_stabilized
It works on Gazebo.
But, there are problem on TF tree...

File: fr01_description/robots/fr01.urdf.xacro (robot description, xacro)
@@ -10,16 +10,15 @@
   <xacro:property name="wheel_width" value="0.16"/>
   <!--==================== Link & Joint ====================-->
+  <!-- Body -->
   <link name="base_footprint"/>
-  <joint name="base_footprint_joint" type="fixed">
+  <xacro:base_stabilized_v0 parent="base_footprint">
+	<origin xyz="0 0 0" rpy="0 0 ${-M_PI/2}"/>
 	<origin xyz="0 0 0.370" rpy="0 0 0"/>
-	<parent link="base_footprint"/>
-	<child link="stabilized_base_link"/>
-  </joint>
-  <!-- Body -->
-  <link name="stabilized_base_link"/>
-  <xacro:base_v0 parent="stabilized_base_link">
+  </xacro:base_stabilized_v0>
+  <xacro:base_link_v0 parent="base_stabilized">
 	<origin xyz="0 0 0" rpy="0 0 ${-M_PI/2}"/>
 	<origin xyz="0 0 0" rpy="0 0 0"/>
-  </xacro:base_v0>
+	<axis xyz="1 1 0"/>
+  </xacro:base_link_v0>
   <!-- Rocker -->
   <xacro:rocker_v0 side="right" parent="base_link">
@@ -153,5 +152,6 @@
   <xacro:wheel_gazebo_v0 part="left_back"/>
   <!-- Body -->
-  <xacro:body_gazebo_vo/>
+  <xacro:base_link_gazebo_v0/>
+  <xacro:base_stabilized_gazebo_v0/>
   <!-- Rocker -->
   <xacro:rocker_gazebo_v0 side="right"/>

File: fr01_description/urdf/body/body.gazebo.xacro (robot description, xacro)
@@ -1,5 +1,5 @@
 <?xml version="1.0"?>
 <robot xmlns:xacro="http://ros.org/wiki/xacro">
-  <xacro:macro name="base_gazebo_v0">
+  <xacro:macro name="base_link_gazebo_v0">
 	<gazebo reference="base_link">
 	  <selfCollide>true</selfCollide>
@@ -8,3 +8,10 @@
     </gazebo>
   </xacro:macro>
+  <xacro:macro name="base_stabilized_gazebo_v0">
+	<gazebo reference="base_stabilized">
+	  <selfCollide>false</selfCollide>
+      <mu1 value="0.8" />
+      <mu2 value="0.8" />
+    </gazebo>
+  </xacro:macro>
 </robot>

File: fr01_description/urdf/body/body.urdf.xacro (robot description, xacro)
@@ -2,10 +2,10 @@
 <robot xmlns:xacro="http://ros.org/wiki/xacro">
   <xacro:include filename="$(find fr01_description)/urdf/body/body.gazebo.xacro"/>
-  <xacro:macro name="base_v0" params="parent *link_origin *joint_origin">
+  <xacro:macro name="base_link_v0" params="parent *link_origin *joint_origin *joint_axis">
 	<joint name="base_link_joint" type="continuous">
-      <insert_block name="joint_origin" />
-      <parent link="${parent}"/>
-      <child link="base_link"/>
-	  <axis xyz="1 1 0"/>
+	  <insert_block name="joint_origin" />
+	  <parent link="${parent}"/>
+	  <child link="base_link"/>
+	  <insert_block name="joint_axis"/>
 	</joint>
     <link name="base_link">
@@ -30,3 +30,25 @@
     </link>
   </xacro:macro>
+  <xacro:macro name="base_stabilized_v0" params="parent *link_origin *joint_origin">
+	<joint name="base_stabilized_joint" type="fixed">
+      <insert_block name="joint_origin" />
+      <parent link="${parent}"/>
+      <child link="base_stabilized"/>
+	</joint>
+    <link name="base_stabilized">
+      <collision>
+		<insert_block name="link_origin"/>
+		<visual/>
+        <geometry>
+		  <mesh filename="package://fr01_description/meshes/collision/base_link.stl"/>
+        </geometry>
+      </collision>
+      <inertial>
+        <mass value="6.441"/>
+        <inertia ixx="0.004" ixy="0.000000000792" ixz="-0.000000001557"
+				 iyy="0.002" iyz="-0.0000000001274"
+				 izz="0.005" />
+      </inertial>
+    </link>
+  </xacro:macro>
 </robot>

Commit message: add transmission of base_link

File: fr01_description/robots/fr01.urdf.xacro (robot description, xacro)
@@ -120,4 +120,6 @@
   </xacro:wheel_v0>
   <!--==================== Transmission ====================-->
+  <!-- base_link -->
+  <xacro:base_link_trans_v0 />
   <!-- Rocker -->
   <xacro:rocker_trans_v0 side="right"/>

File: fr01_description/urdf/body/body.urdf.xacro (robot description, xacro)
@@ -3,13 +3,13 @@
   <xacro:include filename="$(find fr01_description)/urdf/body/body.gazebo.xacro"/>
   <xacro:macro name="base_link_v0" params="parent *link_origin *joint_origin *joint_axis">
-	<joint name="base_link_joint" type="continuous">
-	  <insert_block name="joint_origin" />
-	  <parent link="${parent}"/>
-	  <child link="base_link"/>
-	  <insert_block name="joint_axis"/>
-	</joint>
+    <joint name="base_link_joint" type="continuous">
+      <insert_block name="joint_origin" />
+      <parent link="${parent}"/>
+      <child link="base_link"/>
+      <insert_block name="joint_axis"/>
+    </joint>
     <link name="base_link">
       <visual>
-		<insert_block name="link_origin"/>
+	<insert_block name="link_origin"/>
         <geometry>
           <mesh filename="package://fr01_description/meshes/visual/base_link.dae"/>
@@ -17,7 +17,7 @@
       </visual>
       <collision>
-		<insert_block name="link_origin"/>
+	<insert_block name="link_origin"/>
         <geometry>
-		  <mesh filename="package://fr01_description/meshes/collision/base_link.stl"/>
+	  <mesh filename="package://fr01_description/meshes/collision/base_link.stl"/>
         </geometry>
       </collision>
@@ -25,21 +25,21 @@
         <mass value="6.441"/>
         <inertia ixx="0.004" ixy="0.000000000792" ixz="-0.000000001557"
-				 iyy="0.002" iyz="-0.0000000001274"
-				 izz="0.005" />
+		 iyy="0.002" iyz="-0.0000000001274"
+		 izz="0.005" />
       </inertial>
     </link>
   </xacro:macro>
   <xacro:macro name="base_stabilized_v0" params="parent *link_origin *joint_origin">
-	<joint name="base_stabilized_joint" type="fixed">
+    <joint name="base_stabilized_joint" type="fixed">
       <insert_block name="joint_origin" />
       <parent link="${parent}"/>
       <child link="base_stabilized"/>
-	</joint>
+    </joint>
     <link name="base_stabilized">
       <collision>
-		<insert_block name="link_origin"/>
-		<visual/>
+	<insert_block name="link_origin"/>
+	<visual/>
         <geometry>
-		  <mesh filename="package://fr01_description/meshes/collision/base_link.stl"/>
+	  <mesh filename="package://fr01_description/meshes/collision/base_link.stl"/>
         </geometry>
       </collision>
@@ -47,6 +47,6 @@
         <mass value="6.441"/>
         <inertia ixx="0.004" ixy="0.000000000792" ixz="-0.000000001557"
-				 iyy="0.002" iyz="-0.0000000001274"
-				 izz="0.005" />
+		 iyy="0.002" iyz="-0.0000000001274"
+		 izz="0.005" />
       </inertial>
     </link>

File: fr01_description/urdf/leg/leg.transmission.xacro (robot description, xacro)
@@ -2,14 +2,14 @@
 <robot xmlns:xacro="http://ros.org/wiki/xacro">
   <xacro:macro name="bogie_trans_v0" params="side">
-	<transmission name="bogie_${side}_trans">
+    <transmission name="bogie_${side}_trans">
       <type>transmission_interface/SimpleTransmission</type>
       <joint name="bogie_${side}_joint">
-		<hardwareInterface>EffortJointInterface</hardwareInterface>
+	<hardwareInterface>EffortJointInterface</hardwareInterface>
       </joint>
 	  <actuator name="bogie_${side}_motor">
-		<hardwareInterface>EffortJointInterface</hardwareInterface>
-		<mechanicalReduction>1</mechanicalReduction>
+	    <hardwareInterface>EffortJointInterface</hardwareInterface>
+	    <mechanicalReduction>1</mechanicalReduction>
       </actuator>
-	</transmission>
+    </transmission>
   </xacro:macro>
   <xacro:macro name="rocker_trans_v0" params="side">

Commit message: fix rotatable axis for base_link joint

File: fr01_description/robots/fr01.urdf.xacro (robot description, xacro)
@@ -19,5 +19,5 @@
 	<origin xyz="0 0 0" rpy="0 0 ${-M_PI/2}"/>
 	<origin xyz="0 0 0" rpy="0 0 0"/>
-	<axis xyz="1 1 0"/>
+	<axis xyz="0 1 0"/>
   </xacro:base_link_v0>
   <!-- Rocker -->

Commit message: add hokuyo3d sensor to gazebo and visualize

File: fr01_description/robots/fr01.urdf.xacro (robot description, xacro)
@@ -24,7 +24,7 @@
   <xacro:rocker_v0 side="right" parent="base_link">
   	<origin xyz="0 0 0" rpy="0 0 0"/>
-	<inertia ixx="0.0002582" ixy="-0.0000001417" ixz="-0.00004954"
-			 iyy="0.0004952" iyz="0.00000007736"
-			 izz="0.0003856"/>
+	<inertia ixx="0.001" ixy="-0.0000001417" ixz="-0.00004954"
+		 iyy="0.001" iyz="0.00000007736"
+		 izz="0.001"/>
   	<origin xyz="0 -0.213 0.028 " rpy="0 0 0"/>
 	<axis xyz="0 1 0"/>
@@ -32,7 +32,7 @@
   <xacro:rocker_v0 side="left" parent="base_link">
   	<origin xyz="0 0 0" rpy="0 0 0"/>
-	<inertia ixx="0.0002507" ixy="0.0000001419" ixz="-0.00004954"
-			 iyy="0.0004952" iyz="-0.0004669"
-			 izz="0.0003932"/>
+	<inertia ixx="0.001" ixy="0.0000001419" ixz="-0.00004954"
+		 iyy="0.001" iyz="-0.0004669"
+		 izz="0.001"/>
   	<origin xyz="0 0.213 0.028 " rpy="0 0 0"/>
 	<axis xyz="0 1 0"/>
@@ -42,6 +42,6 @@
   	<origin xyz="0 0 0" rpy="0 0 0"/>
   	<inertia ixx="0.002" ixy="0.0000006258" ixz="-0.000002349"
-  			 iyy="0.002" iyz="-0.0000001149"
-  			 izz="0.003"/>
+  		 iyy="0.002" iyz="-0.0000001149"
+  		 izz="0.003"/>
   	<origin xyz="0.2 -0.019945 -0.15" rpy="0 0 ${M_PI}"/>
   	<axis xyz="0 1 0"/>
@@ -50,6 +50,6 @@
   	<origin xyz="0 0 0" rpy="0 0 0"/>
   	<inertia ixx="0.002" ixy="-0.0000006528" ixz="-0.000002349"
-  			 iyy="0.002" iyz="0.0000001156"
-  			 izz="0.003"/>
+  		 iyy="0.002" iyz="0.0000001156"
+  		 izz="0.003"/>
   	<origin xyz="0.2 0.019945 -0.15" rpy="0 0 ${M_PI}"/>
   	<axis xyz="0 1 0"/>

File: fr01_description/robots/fr01_with_hokuyo3d.urdf.xacro (robot description, xacro)
@@ -9,9 +9,9 @@
   <!-- Joint -->
   <joint name="joint_hokuyo3d" type="fixed">
-    <origin rpy="${M_PI} 0 0" xyz="0.315 0 0.835"/>
-    <parent link="base_footprint"/>
+    <origin rpy="${M_PI/2} 0 0" xyz="0.3405 0 0.463"/>
+    <parent link="base_link"/>
     <child link="hokuyo3d_link"/>
   </joint>
   <!-- Gazebo -->
-  <!-- <xacro:hokuyo3d_gazebo name="hokuyo3d"/> -->
+  <xacro:hokuyo3d_gazebo/>
 </robot>

File: fr01_description/urdf/body/body.urdf.xacro (robot description, xacro)
@@ -25,6 +25,6 @@
       <inertial>
         <mass value="6.441"/>
-        <inertia ixx="0.004" ixy="0.000000000792" ixz="-0.000000001557"
-		 iyy="0.002" iyz="-0.0000000001274"
+        <inertia ixx="0.004" ixy="0.0" ixz="0.0"
+		 iyy="0.002" iyz="0.0"
 		 izz="0.005" />
       </inertial>
@@ -47,6 +47,6 @@
       <inertial>
         <mass value="6.441"/>
-        <inertia ixx="0.004" ixy="0.000000000792" ixz="-0.000000001557"
-		 iyy="0.002" iyz="-0.0000000001274"
+        <inertia ixx="0.004" ixy="0.0" ixz="0.00"
+		 iyy="0.002" iyz="0.0"
 		 izz="0.005" />
       </inertial>

File: fr01_description/urdf/sensor/hokuyo3d.urdf.xacro (robot description, xacro)
@@ -1,22 +1,24 @@
 <?xml version="1.0"?>
 <robot xmlns:xacro="http://ros.org/wiki/xacro">
+  <xacro:include filename="$(find fr01_description)/urdf/sensor/hokuyo3d.gazebo.xacro"/>
   <xacro:macro name="hokuyo3d_link_base_link" params="name">
     <link name="${name}">
       <visual>
         <geometry>
-		  <box size="0.106 0.085 0.105"/>
+	  <!-- <box size="0.106 0.085 0.105"/> -->
+	  <mesh filename="package://fr01_description/meshes/visual/yvt-x002.stl"/>
         </geometry>
       </visual>
       <collision>
-		<origin xyz="0 0 0"/>
+	<origin xyz="0 0 0"/>
         <geometry>
-		  <box size="0.106 0.085 0.105"/>
+	  <box size="0.106 0.085 0.105"/>
         </geometry>
       </collision>
       <inertial>
-        <mass value="0.935"/>
-        <inertia ixx="0.0053937" ixy="0" ixz="0"
-				 iyy="0.00085311" iyz="0"
-				 izz="0.00519899" />
+        <mass value="0.0"/>
+        <inertia ixx="0.016" ixy="-0.006" ixz="-0.00002"
+		 iyy="0.004" iyz="0"
+		 izz="0.018" />
       </inertial>
     </link>
