Commit message: fix hokuyo3d position and shape

File: fr01_description/robots/fr01_with_hokuyo3d.urdf.xacro (robot description, xacro)
@@ -9,5 +9,5 @@
   <!-- Joint -->
   <joint name="joint_hokuyo3d" type="fixed">
-    <origin rpy="${M_PI} 0 0" xyz="0.285 0 0.79"/>
+    <origin rpy="${M_PI} 0 0" xyz="0.315 0 0.835"/>
     <parent link="base_footprint"/>
     <child link="hokuyo3d_link"/>

File: fr01_description/urdf/sensor/hokuyo3d.urdf.xacro (robot description, xacro)
@@ -5,5 +5,5 @@
       <visual>
         <geometry>
-		  <box size="0.085 0.106 0.105"/>
+		  <box size="0.106 0.085 0.105"/>
         </geometry>
       </visual>
@@ -11,5 +11,5 @@
 		<origin xyz="0 0 0"/>
         <geometry>
-		  <box size="0.085 0.106 0.105"/>
+		  <box size="0.106 0.085 0.105"/>
         </geometry>
       </collision>

Commit message: update sensor position param

File: fr01_description/robots/fr01_with_hokuyo3d.urdf.xacro (robot description, xacro)
@@ -9,6 +9,6 @@
   <!-- Joint -->
   <joint name="joint_hokuyo3d" type="fixed">
-    <origin rpy="${M_PI} 0 0" xyz="0.315 0 0.835"/>
-    <parent link="base_footprint"/>
+    <origin rpy="${M_PI} 0 0" xyz="0.315 0 0.435"/>
+    <parent link="base_stabilized"/>
     <child link="hokuyo3d_link"/>
   </joint>

Commit message: fixed rotation of hokuyo3d

File: fr01_description/robots/fr01_with_hokuyo3d.urdf.xacro (robot description, xacro)
@@ -9,5 +9,5 @@
   <!-- Joint -->
   <joint name="joint_hokuyo3d" type="fixed">
-    <origin rpy="${M_PI/2} 0 0" xyz="0.3405 0 0.463"/>
+    <origin rpy="0 0 0" xyz="0.3405 0 0.463"/>
     <parent link="base_link"/>
     <child link="hokuyo3d_link"/>

Commit message: inversed hokuyo3d for tf

File: fr01_description/robots/fr01_with_hokuyo3d.urdf.xacro (robot description, xacro)
@@ -9,5 +9,5 @@
   <!-- Joint -->
   <joint name="joint_hokuyo3d" type="fixed">
-    <origin rpy="0 0 0" xyz="0.3405 0 0.463"/>
+    <origin rpy="${M_PI} 0 0" xyz="0.3405 0 0.463"/>
     <parent link="base_link"/>
     <child link="hokuyo3d_link"/>
