Commit message: add camera setting

File: fr01_description/robots/fr01_with_sensors.urdf.xacro (robot description, xacro)
@@ -2,4 +2,5 @@
 <robot name="fr01" xmlns:xacro="http://ros.org/wiki/xacro">
   <!-- File Include -->
+  <xacro:include filename="$(find fr01_description)/urdf/sensor/c930.urdf.xacro" />
   <xacro:include filename="$(find fr01_description)/urdf/sensor/hokuyo3d.urdf.xacro"/>
   <xacro:include filename="$(find fr01_description)/robots/fr01.urdf.xacro"/>
@@ -9,7 +10,14 @@
   <!-- Joint -->
   <joint name="joint_hokuyo3d" type="fixed">
-    <origin rpy="${M_PI} 0 0" xyz="0.315 0 0.835"/>
-    <parent link="base_footprint"/>
+    <origin rpy="${M_PI} 0 0" xyz="0.3405 0 0.463"/>
+    <parent link="base_link"/>
     <child link="hokuyo3d_link"/>
+  </joint>
+  <xacro:c930_link_base_link name="c930_link"/>
+  <!-- Joint -->
+  <joint name="joint_c930" type="fixed">
+    <origin rpy="0 0 0" xyz="0.3 0 0.0"/>
+    <parent link="base_link"/>
+    <child link="c930_link"/>
   </joint>
   <!-- Gazebo -->

File: fr01_description/urdf/sensor/c930.urdf.xacro (robot description, xacro)
@@ -15,5 +15,5 @@
       </collision>
       <inertial>
-        <mass value="0.935"/>
+        <mass value="0.0"/>
         <inertia ixx="0.0053937" ixy="0" ixz="0"
 		 iyy="0.00085311" iyz="0"

Commit message: make the camera disable

File: fr01_description/robots/fr01_with_sensors.urdf.xacro (robot description, xacro)
@@ -2,5 +2,5 @@
 <robot name="fr01" xmlns:xacro="http://ros.org/wiki/xacro">
   <!-- File Include -->
-  <xacro:include filename="$(find fr01_description)/urdf/sensor/c930.urdf.xacro" />
+  <!-- <xacro:include filename="$(find fr01_description)/urdf/sensor/c930.urdf.xacro" /> -->
   <xacro:include filename="$(find fr01_description)/urdf/sensor/hokuyo3d.urdf.xacro"/>
   <xacro:include filename="$(find fr01_description)/robots/fr01.urdf.xacro"/>
@@ -14,11 +14,11 @@
     <child link="hokuyo3d_link"/>
   </joint>
-  <xacro:c930_link_base_link name="c930_link"/>
+  <!-- <xacro:c930_link_base_link name="c930_link"/> -->
   <!-- Joint -->
-  <joint name="joint_c930" type="fixed">
-    <origin rpy="0 0 0" xyz="0.3 0 0.0"/>
-    <parent link="base_link"/>
-    <child link="c930_link"/>
-  </joint>
+  <!-- <joint name="joint_c930" type="fixed"> -->
+  <!--   <origin rpy="0 0 0" xyz="0.3 0 0.0"/> -->
+  <!--   <parent link="base_link"/> -->
+  <!--   <child link="c930_link"/> -->
+  <!-- </joint> -->
   <!-- Gazebo -->
   <!-- <xacro:hokuyo3d_gazebo name="hokuyo3d"/> -->
