Commit message: add dae file of hokuyo3d

File: fr01_description/urdf/sensor/hokuyo3d.urdf.xacro (robot description, xacro)
@@ -7,5 +7,5 @@
         <geometry>
 	  <!-- <box size="0.106 0.085 0.105"/> -->
-	  <mesh filename="package://fr01_description/meshes/visual/yvt-x002.stl"/>
+	  <mesh filename="package://fr01_description/meshes/visual/yvt-x002.dae"/>
         </geometry>
       </visual>

Commit message: delete unused codes and white spaces

File: fr01_description/urdf/sensor/hokuyo3d.urdf.xacro (robot description, xacro)
@@ -6,5 +6,4 @@
       <visual>
         <geometry>
-	  <!-- <box size="0.106 0.085 0.105"/> -->
 	  <mesh filename="package://fr01_description/meshes/visual/yvt-x002.dae"/>
         </geometry>
